Commit message: update urdf limit accroding to calibrate of real arm

File: src/lerobot_description/urdf/so101.urdf.xacro (robot description, xacro)
@@ -1,4 +1,5 @@
 <?xml version="1.0"?>
-<robot name="so101" xmlns:xacro="http://www.ros.org/wiki/xacro">
+<robot xmlns:xacro="http://www.ros.org/wiki/xacro" name="so101">
+    <xacro:arg name="use_sim" default="true"/>
     <xacro:include filename="$(find lerobot_description)/urdf/so101_base.xacro" />
     <xacro:include filename="$(find lerobot_description)/urdf/so101_gazebo.xacro" />

File: src/lerobot_description/urdf/so101_base.xacro (robot description, xacro)
@@ -345,5 +345,6 @@
 		<child link="jaw" />
 		<axis xyz="0 0 1" />
-		<limit effort="10" velocity="10" lower="-0.174533" upper="1.74533" />
+		<!-- calibrated limits: raw(2041,3457) home(2749) = (-1.0858,+1.0858) rad -->
+		<limit effort="10" velocity="10" lower="-1.0858" upper="1.0858"/>
 	</joint>
 	<transmission name="6_trans">
@@ -363,5 +364,6 @@
 		<child link="gripper" />
 		<axis xyz="0 0 1" />
-		<limit effort="10" velocity="10" lower="-2.79253" upper="2.79253" />
+		<!-- calibrated limits: raw(64,3860) home(1962) = (-2.9115,+2.9115) rad -->
+		<limit effort="10" velocity="10" lower="-2.9115" upper="2.9115" />
 	</joint>
 	<transmission name="5_trans">
@@ -399,5 +401,6 @@
 		<child link="lower_arm" />
 		<axis xyz="0 0 1" />
-		<limit effort="10" velocity="10" lower="-1.74533" upper="1.5708" />
+		<!-- calibrated limits: raw(755,2948) home(1851) = (-1.6813,+1.6828) rad -->
+		<limit effort="10" velocity="10" lower="-1.6813" upper="1.6828" />
 	</joint>
 	<transmission name="3_trans">
@@ -435,5 +438,6 @@
 		<child link="shoulder" />
 		<axis xyz="0 0 1" />
-		<limit effort="10" velocity="10" lower="-1.91986" upper="1.91986" />
+		<!-- calibrated limits: raw(817,3516) home(2166) = (-2.0693,+2.0709) rad -->
+		<limit effort="10" velocity="10" lower="-2.0693" upper="2.0709" />
 	</joint>
 	<transmission name="1_trans">

File: src/lerobot_description/urdf/so101_ros2_control.xacro (robot description, xacro)
@@ -1,13 +1,22 @@
 <?xml version="1.0"?>
 <robot xmlns:xacro="http://www.ros.org/wiki/xacro">
+    <xacro:arg name="use_sim" default="true"/>
     <ros2_control name="RobotSystem" type="system">
-        <!-- ros2_control Gazebo -->
-        <hardware>
-            <plugin>gz_ros2_control/GazeboSimSystem</plugin>
-        </hardware>
+        <xacro:if value="$(arg use_sim)">
+            <hardware>
+                <plugin>gz_ros2_control/GazeboSimSystem</plugin>
+            </hardware>
+        </xacro:if>
+        <xacro:unless value="$(arg use_sim)">
+            <hardware>
+                <plugin>topic_based_ros2_control/TopicBasedSystem</plugin>
+                <param name="joint_commands_topic">/so101_follower/joint_commands</param>
+                <param name="joint_states_topic">/so101_follower/joint_states</param>
+            </hardware>
+        </xacro:unless>
         <joint name="1">
             <command_interface name="position">
-                <param name="min">-1.91986</param>
-                <param name="max">1.91986</param>
+                <param name="min">-2.0693</param>
+                <param name="max">2.0709</param>
             </command_interface>
             <state_interface name="position" />
@@ -22,6 +31,6 @@
         <joint name="3">
             <command_interface name="position">
-                <param name="min">-1.74533</param>
-                <param name="max">1.5708</param>
+                <param name="min">-1.6813</param>
+                <param name="max">1.6828</param>
             </command_interface>
             <state_interface name="position" />
@@ -36,6 +45,6 @@
         <joint name="5">
             <command_interface name="position">
-                <param name="min">-2.79253</param>
-                <param name="max">2.79253</param>
+                <param name="min">-2.9115</param>
+                <param name="max">2.9115</param>
             </command_interface>
             <state_interface name="position" />
@@ -43,6 +52,6 @@
         <joint name="6">
             <command_interface name="position">
-                <param name="min">-0.174533</param>
-                <param name="max">1.74533</param>
+                <param name="min">-1.0858</param>
+                <param name="max">1.0858</param>
             </command_interface>
             <state_interface name="position" />
